File: wled_esp8266/wled_esp8266.kicad_pcb (KiCad board)
At the start: 2 copper layers, 34 parts, among them J1 PWR, J2 Conn_01x05, J3 Screw_Terminal_01x04, J4 LED_STRIPT, J5 USB_B_Micro, Q1 IRF3708, Q2 IRF3708, Q3 IRF3708, U1 ESP-12F, U2 AMS1117-3.3

Commit message: update new pcb
Parts:
- removed C1, C3, C4, C6: 100nF, Capacitor_SMD:C_0805_2012Metric_Pad1.18x1.45mm_HandSolder
- removed C5: 100uF, Capacitor_Tantalum_SMD:CP_EIA-3528-12_Kemet-T_Pad1.50x2.35mm_HandSolder
- removed D1, D2: LED, LED_SMD:LED_0805_2012Metric_Pad1.15x1.40mm_HandSolder
- removed J2: Conn_01x05, Connector_PinSocket_2.54mm:PinSocket_1x05_P2.54mm_Vertical
- removed J5: USB_B_Micro, Connector_USB:USB_Micro
- removed R1, R2, R3, R4, R5: 12K, Resistor_SMD:R_0805_2012Metric_Pad1.20x1.40mm_HandSolder
- removed R6: 220, Resistor_SMD:R_0805_2012Metric_Pad1.20x1.40mm_HandSolder
- removed R7: 330, Resistor_SMD:R_0805_2012Metric_Pad1.20x1.40mm_HandSolder
- removed U2: AMS1117-3.3, Package_TO_SOT_SMD:SOT-223-3_TabPin2
- C2, C7, D3, R12, R8: moved to F.Cu
- U1: value ESP-12F -> ESP8266Nodemcu; footprint RF_Module:ESP-12E -> Module:ESP8266Nodemcu
- moved C2 92.8 mm to (191.2, 75.7), turned to 0 degrees
- moved Q3 80.3 mm to (182.7, 78.2), turned to 0 degrees
- moved R11 79.2 mm to (191.2, 78.7)
- moved R9 62.3 mm to (186.1, 83.7), turned to 0 degrees
- moved Q1 60.5 mm to (177.6, 87.3), turned to 0 degrees
- moved J3 60.1 mm to (158.2, 78.7), turned to 0 degrees
- moved C8 58.5 mm to (173.9, 92.8), turned to 0 degrees
- moved J1 57.3 mm to (158.1, 87.8), turned to 0 degrees
- moved R10 39.4 mm to (166.7, 102.8)
- moved MIC1 33.6 mm to (157.2, 103.7), turned to 0 degrees
- moved J4 18.6 mm to (158.1, 96.8), turned to 0 degrees
- moved U1 15.6 mm to (140.4, 99.1)
- moved D3 15.4 mm to (140.4, 125.5)
- moved C7 15.0 mm to (161.9, 102.8), turned to 0 degrees
- moved R12 11.7 mm to (145.2, 125.5), turned to 0 degrees
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Connections:
- U1 pad 1: RST -> +5V
- U1 pad 13: (no net) -> unconnected-(U1-Pad13)
- U1 pad 15: GND -> MICRO
- U1 pad 16: GPIO15 -> unconnected-(U1-Pad16)
- U1 pad 17: GPIO2 -> unconnected-(U1-Pad17)
- U1 pad 18: GPIO0 -> unconnected-(U1-Pad18)
- U1 pad 19: R_LED -> unconnected-(U1-Pad19)
- U1 pad 2: MICRO -> GND
- U1 pad 20: B_LED -> unconnected-(U1-Pad20)
- U1 pad 21: RX -> unconnected-(U1-Pad21)
- U1 pad 22: TX -> unconnected-(U1-Pad22)
- U1 pad 3: EN -> unconnected-(U1-Pad3)
- U1 pad 5: G_LED -> +3V3
- U1 pad 8: +3V3 -> unconnected-(U1-Pad8)
Routing:
- net +3V3: track 40.0 -> 0.00 mm, vias 3 -> 0
- net GPIO0: track 31.0 -> 0.00 mm, vias 1 -> 0
- net BLUE: track 30.4 -> 0.00 mm, vias 5 -> 0
- net B_LED: track 27.8 -> 0.00 mm, vias 2 -> 0
- net RX: track 24.1 -> 0.00 mm
- net TX: track 22.8 -> 0.00 mm
- net GREEN: track 20.9 -> 0.00 mm, vias 4 -> 0
- net RST: track 20.8 -> 0.00 mm, vias 1 -> 0
- net R_LED: track 19.9 -> 0.00 mm
- net G_LED: track 19.3 -> 0.00 mm
- net MICRO: track 16.4 -> 0.00 mm
- net GPIO2: track 12.6 -> 0.00 mm, vias 1 -> 0
- net RED: track 11.2 -> 0.00 mm
- net EN: track 3.73 -> 0.00 mm, vias 1 -> 0
- net GPIO15: track 2.84 -> 0.00 mm, vias 1 -> 0

Commit message: update PCB
Parts:
- removed C7: 100nF, Capacitor_SMD:C_0805_2012Metric_Pad1.18x1.45mm_HandSolder
- removed R12: 220, Resistor_SMD:R_0805_2012Metric_Pad1.20x1.40mm_HandSolder
- added C1: 100nF, Capacitor_SMD:C_0805_2012Metric_Pad1.18x1.45mm_HandSolder, B.Cu at (118.5, 109.5)
- added C3: 100nF, Capacitor_SMD:C_0805_2012Metric_Pad1.18x1.45mm_HandSolder, B.Cu at (112.5, 134.5)
- added D1: LED, LED_THT:LED_D3.0mm, F.Cu at (124.1, 96.8)
- added J2: USB_A_Stacked, Connector_USB:USB_A_Wuerth_61400826021_Horizontal_Stacked, F.Cu at (122.4, 115.6)
- added J5: Conn_01x02, Connector_PinSocket_2.54mm:PinSocket_1x02_P2.54mm_Vertical, F.Cu at (75.9, 110.0)
- added J6: Conn_01x02, Connector_PinSocket_2.54mm:PinSocket_1x02_P2.54mm_Vertical, F.Cu at (117.7, 116.5)
- added J7: Conn_01x02, Connector_PinSocket_2.54mm:PinSocket_1x02_P2.54mm_Vertical, F.Cu at (105.0, 133.7)
- added R1: 330, Resistor_SMD:R_0805_2012Metric_Pad1.20x1.40mm_HandSolder, B.Cu at (119.1, 96.9)
- C2, C8, R10, R11, R8, R9: moved to B.Cu
- D3: footprint LED_SMD:LED_0805_2012Metric_Pad1.15x1.40mm_HandSolder -> LED_THT:LED_D3.0mm
- J4: value LED_STRIPT -> USB_A_Stacked; footprint TerminalBlock:TerminalBlock_bornier-3_P5.08mm -> Connector_USB:USB_A_Wuerth_61400826021_Horizontal_Stacked
- Q1, Q2, Q3: footprint Package_TO_SOT_SMD:TO-252-3_TabPin4 -> Package_TO_SOT_SMD:TO-252-2; moved to B.Cu
- U1: footprint Module:ESP8266Nodemcu -> Module:LoLinNodeMcu(esp8266)
- moved R9 117.9 mm to (76.2, 126.4)
- moved C2 117.2 mm to (77.7, 104.9)
- moved Q1 111.6 mm to (76.1, 133.6), turned to -90 degrees
- moved R11 110.6 mm to (91.4, 126.3)
- moved Q3 106.9 mm to (91.4, 133.7), turned to -90 degrees
- moved J3 105.1 mm to (76.1, 144.4)
- moved C8 96.7 mm to (77.9, 82.0), turned to -90 degrees
- moved MIC1 86.6 mm to (74.5, 77.9)
- moved R10 86.2 mm to (83.8, 126.4)
- moved J1 83.1 mm to (75.1, 90.4), turned to -90 degrees
- moved J4 66.6 mm to (106.5, 138.9)
- moved U1 58.8 mm to (83.4, 114.0)
- moved Q2 48.5 mm to (83.8, 133.7), turned to -90 degrees
- moved R8 41.8 mm to (118.9, 92.7), turned to 180 degrees
- moved D3 37.0 mm to (124.0, 92.4), turned to 90 degrees
Connections:
- J4 pad 1: Net-(J4-Pad1) -> Net-(C3-Pad1)
- J4 pad 2: +5V -> unconnected-(J4-Pad2)
- J4 pad 3: GND -> unconnected-(J4-Pad3)
- MIC1 pad 2: GND -> +3V3
- MIC1 pad 3: +3V3 -> GND
- Q1 pad 2: unconnected-(Q1-Pad2) -> RED
- Q2 pad 2: unconnected-(Q2-Pad2) -> GREEN
- Q3 pad 2: unconnected-(Q3-Pad2) -> BLUE
- U1 pad 1: +5V -> Net-(J5-Pad1)
- U1 pad 17: unconnected-(U1-Pad17) -> GND
- U1 pad 26: GPIO2 -> unconnected-(U1-Pad26)
Other:
- board outline added: 62.8 x 80 mm
